Commit message: [Stash] Apply all changes. corrected hardware from problem of last commit

File: phantom_control/description/physical_phantom.ros2_control.xacro (robot description, xacro)
@@ -6,5 +6,4 @@
         <plugin>phantom_control/PhantomPincherSystem</plugin>
            <param name="device_name">/dev/tty.usbserial-FT5WIT8G</param>
-           <!-- <param name="baud_rate">1000000</param> -->
           <!--  -->
       </hardware>

File: phantom_description/urdf/turtlebot_arm.urdf.xacro (robot description, xacro)
@@ -13,10 +13,11 @@
     <xacro:property name="wrist_llimit" value="-1.745"/>
     <xacro:property name="wrist_ulimit" value="1.745"/>
+    <xacro:arg name="phantom_x_100" default="true"/>
+    <xacro:property name="phantom_x_100" value="$(arg phantom_x_100)"/>
     <!-- Included URDF Files -->
     <xacro:include filename="$(find phantom_description)/urdf/turtlebot_arm.xacro"/>
     <!-- <xacro:include filename="$(find phantom_control)/description/phantom.ros2_control.xacro"/> -->
     <xacro:include filename="$(find phantom_control)/description/physical_phantom.ros2_control.xacro"/>
-    <xacro:call macro="phantom_ros2_control" name="turtlebot_arm" prefix="">
-    </xacro:call>
+    <xacro:call macro="phantom_ros2_control" name="turtlebot_arm" prefix=""/>
     <!-- As we don't have here a turtlebot base, add a base_link link as its location reference -->
     <link name="base_link"/>
@@ -26,5 +27,5 @@
     <!-- Turtlebot arm macro -->
     <xacro:call macro="turtlebot_arm" parent="arm_mount_link" color="Black" gripper_color="Black"
-                    pincher_gripper="true" turtlebot_gripper="false">
+                    pincher_gripper="true" turtlebot_gripper="false" phantom_x_100="${phantom_x_100}">
       <!-- Place the "floating" arm at the location it should be if mounted on a turtlebot,
            as pick and place and other demos assume this location -->

File: phantom_description/urdf/turtlebot_arm.xacro (robot description, xacro)
@@ -15,5 +15,5 @@
     <color rgba="0.22 0.32 0.14 1.0"/>
   </material>
-  <xacro:macro name="turtlebot_arm" params="parent color pincher_gripper turtlebot_gripper gripper_color *origin">
+  <xacro:macro name="turtlebot_arm" params="parent color pincher_gripper turtlebot_gripper gripper_color phantom_x_100 *origin">
     <link name="arm_base_link"/>
     <joint name="arm_base_joint" type="fixed">
@@ -62,7 +62,12 @@
     </xacro:call >
     <!-- elbow joint -->
-    <xacro:call macro="dynamixel_AX12_fixed" parent="arm_shoulder_F3_0_link" name="arm_elbow_flex_servo">
-      <origin xyz="0 0 ${-AX12_HEIGHT-F10_HEIGHT+0.001}" rpy="0 ${M_PI} 0"/>
-    </xacro:call >
+      <xacro:call macro="dynamixel_AX12_fixed" parent="arm_shoulder_F3_0_link" name="arm_elbow_flex_servo">
+      <xacro:if value="${phantom_x_100}">
+        <origin xyz="0 0 ${-AX12_HEIGHT-F10_HEIGHT+0.001}" rpy="0 0 0"/>
+      </xacro:if>
+      <xacro:if value="${not phantom_x_100}">
+        <origin xyz="0 0 ${-AX12_HEIGHT-F10_HEIGHT+0.001}" rpy="0 ${M_PI} 0"/>
+      </xacro:if>
+      </xacro:call >
     <xacro:call macro="bioloid_F4_revolute" parent="arm_elbow_flex_servo_link" name="arm_elbow_flex" color="${color}"
                          vlimit="${joints_vlimit}" llimit="${elbow_llimit}" ulimit="${elbow_ulimit}">
