Commit message: [Update] Rviz digital twin. Joint Broadcaster for waist, shoulder, elbow and wrist_angle. No controller

File: phantom_description/urdf/px100/px100.urdf.xacro (robot description, xacro)
@@ -46,5 +46,5 @@
   <joint name="waist" type="revolute">
     <axis xyz="0 0 1"/>
-    <limit effort="1" lower="${-pi + pi_offset}" upper="${pi - pi_offset}" velocity="${pi}"/>
+    <limit effort="1" lower="${0 + pi_offset}" upper="${2 * pi - pi_offset}" velocity="${pi}"/>
     <origin rpy="0 0 0" xyz="0 0 0.05085"/>
     <parent link="$(arg robot_name)/$(arg base_link_frame)"/>
@@ -82,7 +82,7 @@
   </link>
   <joint name="shoulder" type="revolute">
-    <axis xyz="0 1 0"/>
-    <limit effort="2" lower="${radians(-111)}" upper="${radians(107)}" velocity="${pi}"/>
-    <origin rpy="0 0 0" xyz="0 0 0.04225"/>
+    <axis xyz="0 -1 0"/>
+    <limit effort="2" lower="${0 + pi_offset}" upper="${2 * pi - pi_offset}" velocity="${pi}"/>
+    <origin rpy="${pi} 0 0" xyz="0 0 0.04225"/>
     <parent link="$(arg robot_name)/shoulder_link"/>
     <child link="$(arg robot_name)/upper_arm_link"/>
@@ -120,6 +120,6 @@
   <joint name="elbow" type="revolute">
     <axis xyz="0 1 0"/>
-    <limit effort="2" lower="${radians(-121)}" upper="${radians(92)}" velocity="${pi}"/>
-    <origin rpy="0 0 0" xyz="0.035 0 0.1"/>
+    <limit effort="2" lower="${0 + pi_offset}" upper="${2 * pi - pi_offset}" velocity="${pi}"/>
+    <origin rpy="0 0 ${pi}" xyz="0.035 0 0.1"/>
     <parent link="$(arg robot_name)/upper_arm_link"/>
     <child link="$(arg robot_name)/forearm_link"/>
@@ -156,7 +156,7 @@
   </link>
   <joint name="wrist_angle" type="revolute">
-    <axis xyz="0 1 0"/>
-    <limit effort="1" lower="${radians(-100)}" upper="${radians(123)}"  velocity="${pi}"/>
-    <origin rpy="0 0 0" xyz="0.1 0 0"/>
+    <axis xyz="0 -1 0"/>
+    <limit effort="1" lower="${0 + pi_offset}" upper="${2 * pi - pi_offset}"   velocity="${pi}"/>
+    <origin rpy="0 0 ${pi}" xyz="0.1 0 0"/>
     <parent link="$(arg robot_name)/forearm_link"/>
     <child link="$(arg robot_name)/gripper_link"/>
